File: kicad_concept/testbed_heatguard.kicad_sch (KiCad schematic)
At the start: 8 parts, among them K1 Guard switch

Commit message: v1.0 as ordered
Other:
- note removed: "Inject Tref short"
Changed lines of the file:
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@@
-		)
-	)
-	(text "Inject Tref short"
-		(exclude_from_sim no)
-		(at 136.398 33.02 0)
-		(effects
-			(font
-				(face "FreeSans")
-				(size 1.27 1.27)
-			)
-			(justify left)
 		)
 	)
